Commit message: 0502 전체 수정 커밋

File: husky/husky_description/urdf/husky.urdf.xacro (robot description, xacro)
@@ -362,18 +362,3 @@
   <!-- Optional for Clearpath internal softwares -->
   <xacro:include filename="$(arg cpr_urdf_extras)" />
-  <!-- ========== OS1-32 LiDAR Sensor ========== -->
-  <link name="os1_lidar">
-    <visual>
-      <geometry>
-        <cylinder radius="0.05" length="0.08"/>
-      </geometry>
-      <material name="Grey"/>
-      <origin xyz="0 0 0" rpy="0 0 0"/>
-    </visual>
-  </link>
-  <joint name="os1_lidar_joint" type="fixed">
-    <parent link="base_link"/>
-    <child link="os1_lidar"/>
-    <origin xyz="0.2 0 0.5" rpy="0 0 0"/>
-  </joint>
 </robot>

Commit message: 0507

File: husky/husky_description/urdf/husky.urdf.xacro (robot description, xacro)
@@ -26,4 +26,23 @@
   <xacro:arg name="imu_rpy"     default="$(optenv HUSKY_IMU_RPY 0 -1.5708 3.1416)"/>
   <xacro:arg name="imu_parent"  default="$(optenv HUSKY_IMU_PARENT base_link)"/>
+  <!-- 2) OS1-64 LiDAR 모델 포함 -->
+  <xacro:include filename="$(find ouster_description)/urdf/OS1-64.urdf.xacro"/>
+  <xacro:OS1-64
+    parent="top_chassis_link"
+    name="os1"
+    topic_points="/os1/points"
+    topic_imu="/os1/imu"
+    hz="10"
+    lasers="64"
+    samples="512"
+    min_range="0.9"
+    max_range="75.0"
+    noise="0.008"
+    lidar_link="os1_lidar"
+    imu_link="os1_imu"
+    vfov_min="-.26"
+    vfov_max=".26">
+    <origin xyz="0 0 0.3" rpy="0 0 0"/>
+  </xacro:OS1-64>
   <!-- LMS1XX Laser Primary and Secondary -->
   <xacro:arg name="laser_enabled"           default="$(optenv HUSKY_LMS1XX_ENABLED 0)" />

File: husky/husky_description/urdf/wheel.urdf.xacro (robot description, xacro)
@@ -1,67 +1,53 @@
 <?xml version="1.0"?>
-<!--
-Software License Agreement (BSD)
-\file      wheel.urdf.xacro
-\authors   Paul Bovbel <pbovbel@clearpathrobotics.com>
-\copyright Copyright (c) 2015, Clearpath Robotics, Inc., All rights reserved.
-Redistribution and use in source and binary forms, with or without modification, are permitted provided that
-the following conditions are met:
- * Redistributions of source code must retain the above copyright notice, this list of conditions and the
-   following disclaimer.
- * Redistributions in binary form must reproduce the above copyright notice, this list of conditions and the
-   following disclaimer in the documentation and/or other materials provided with the distribution.
- * Neither the name of Clearpath Robotics nor the names of its contributors may be used to endorse or promote
-   products derived from this software without specific prior written permission.
-THIS SOFTWARE IS PROVIDED BY THE COPYRIGHT HOLDERS AND CONTRIBUTORS "AS IS" AND ANY EXPRESS OR IMPLIED WAR-
-RANTIES, INCLUDING, BUT NOT LIMITED TO, THE IMPLIED WARRANTIES OF MERCHANTABILITY AND FITNESS FOR A PARTICULAR
-PURPOSE ARE DISCLAIMED. IN NO EVENT SHALL THE COPYRIGHT HOLDER OR CONTRIBUTORS BE LIABLE FOR ANY DIRECT, IN-
-DIRECT, INCIDENTAL, SPECIAL, EXEMPLARY, OR CONSEQUENTIAL DAMAGES (INCLUDING, BUT NOT LIMITED TO, PROCUREMENT
-OF SUBSTITUTE GOODS OR SERVICES; LOSS OF USE, DATA, OR PROFITS; OR BUSINESS INTERRUPTION) HOWEVER CAUSED AND
-ON ANY THEORY OF LIABILITY, WHETHER IN CONTRACT, STRICT LIABILITY, OR TORT (INCLUDING NEGLIGENCE OR OTHERWISE)
-ARISING IN ANY WAY OUT OF THE USE OF THIS SOFTWARE, EVEN IF ADVISED OF THE POSSIBILITY OF SUCH DAMAGE.
--->
-<robot xmlns:xacro="http://ros.org/wiki/xacro" name="husky_wheel">
-	<xacro:macro name="husky_wheel" params="wheel_prefix *joint_pose">
-		<link name="${wheel_prefix}_wheel_link">
-			<inertial>
-				<mass value="2.637" />
-				<origin xyz="0 0 0" />
-				<inertia  ixx="0.02467" ixy="0" ixz="0" iyy="0.04411" iyz="0" izz="0.02467" />
-			</inertial>
-			<visual>
-				<origin xyz="0 0 0" rpy="0 0 0" />
-				<geometry>
-					<mesh filename="package://husky_description/meshes/wheel.dae" />
-				</geometry>
-			</visual>
-			<collision>
-				<origin xyz="0 0 0" rpy="${M_PI/2} 0 0" />
-				<geometry>
-					<cylinder length="${wheel_length}" radius="${wheel_radius}" />
-				</geometry>
-			</collision>
-		</link>
-		<gazebo reference="${wheel_prefix}_wheel_link">
-			<mu1 value="1.0"/>
-			<mu2 value="1.0"/>
-			<kp value="10000000.0" />
-			<kd value="1.0" />
-			<fdir1 value="1 0 0"/>
-		</gazebo>
-		<joint name="${wheel_prefix}_wheel" type="continuous">
-			<parent link="base_link"/>
-			<child link="${wheel_prefix}_wheel_link"/>
-			<xacro:insert_block name="joint_pose"/>
-			<axis xyz="0 1 0" rpy="0 0 0" />
-		</joint>
-		<transmission name="${wheel_prefix}_wheel_trans" type="SimpleTransmission">
-			<type>transmission_interface/SimpleTransmission</type>
-			<actuator name="${wheel_prefix}_wheel_motor">
-				<mechanicalReduction>1</mechanicalReduction>
-			</actuator>
-			<joint name="${wheel_prefix}_wheel">
-				<hardwareInterface>hardware_interface/VelocityJointInterface</hardwareInterface>
-			</joint>
-		</transmission>
-	</xacro:macro>
+<robot xmlns:xacro="http://www.ros.org/wiki/xacro" name="husky_wheel">
+  <xacro:property name="M_PI" value="3.14159"/>
+  <xacro:macro name="husky_wheel" params="wheel_prefix *joint_pose">
+    <!-- 1) Wheel Link -->
+    <link name="${wheel_prefix}_wheel_link">
+      <inertial>
+        <mass value="2.637"/>
+        <origin xyz="0 0 0"/>
+        <inertia ixx="0.02467" ixy="0" ixz="0"
+                 iyy="0.04411" iyz="0" izz="0.02467"/>
+      </inertial>
+      <visual>
+        <origin xyz="0 0 0" rpy="0 0 0"/>
+        <geometry>
+          <mesh filename="package://husky_description/meshes/wheel.dae"/>
+        </geometry>
+      </visual>
+      <collision>
+        <origin xyz="0 0 0" rpy="${M_PI/2} 0 0"/>
+        <geometry>
+          <cylinder length="${wheel_length}" radius="${wheel_radius}"/>
+        </geometry>
+      </collision>
+    </link>
+    <!-- 2) Gazebo friction/ODE params -->
+    <gazebo reference="${wheel_prefix}_wheel_link">
+      <mu1 value="1.0"/>
+      <mu2 value="1.0"/>
+      <kp value="10000000.0"/>
+      <kd value="1.0"/>
+      <fdir1 value="1 0 0"/>
+    </gazebo>
+    <!-- 3) Continuous Joint -->
+    <joint name="${wheel_prefix}_wheel" type="continuous">
+      <parent link="base_link"/>
+      <child link="${wheel_prefix}_wheel_link"/>
+      <xacro:insert_block name="joint_pose"/>
+      <axis xyz="0 1 0"/>
+    </joint>
+    <!-- 4) Transmission with hardwareInterface on both actuator & joint -->
+    <transmission name="${wheel_prefix}_wheel_trans">
+      <type>transmission_interface/SimpleTransmission</type>
+      <actuator name="${wheel_prefix}_wheel_motor">
+        <mechanicalReduction>1</mechanicalReduction>
+        <hardwareInterface>hardware_interface/VelocityJointInterface</hardwareInterface>
+      </actuator>
+      <joint name="${wheel_prefix}_wheel">
+        <hardwareInterface>hardware_interface/VelocityJointInterface</hardwareInterface>
+      </joint>
+    </transmission>
+  </xacro:macro>
 </robot>

Commit message: 0511

File: husky/husky_description/urdf/husky.urdf.xacro (robot description, xacro)
@@ -35,5 +35,5 @@
     hz="10"
     lasers="32"
-    samples="512"
+    samples="1024"
     min_range="0.9"
     max_range="75.0"
@@ -41,7 +41,7 @@
     lidar_link="os1_lidar"
     imu_link="os1_imu"
-    vfov_min="-.26"
-    vfov_max=".26">
-    <origin xyz="0 0 0.3" rpy="0 0 0"/>
+    vfov_min="-.30"
+    vfov_max=".30">
+    <origin xyz="0 0 0.6" rpy="0 0 0"/>
   </xacro:OS1-32>
   <!-- LMS1XX Laser Primary and Secondary -->

Commit message: 0528

File: husky/husky_description/urdf/husky.urdf.xacro (robot description, xacro)
@@ -45,4 +45,20 @@
     <origin xyz="0 0 0.6" rpy="0 0 0"/>
   </xacro:OS1-32>
+    <!-- GPS Link -->
+  <link name="gps_link">
+    <visual>
+      <geometry>
+        <box size="0.05 0.05 0.05"/>
+      </geometry>
+      <material name="Blue">
+        <color rgba="0 0 1 1"/>
+      </material>
+    </visual>
+  </link>
+  <joint name="gps_joint" type="fixed">
+    <parent link="base_link"/>
+    <child link="gps_link"/>
+    <origin xyz="0 0 1.0" rpy="0 0 0"/>
+  </joint>
   <!-- LMS1XX Laser Primary and Secondary -->
   <xacro:arg name="laser_enabled"           default="$(optenv HUSKY_LMS1XX_ENABLED 0)" />
@@ -362,22 +378,26 @@
     </plugin>
   </gazebo>
-  <gazebo>
-    <plugin name="gps_controller" filename="libhector_gazebo_ros_gps.so">
-      <robotNamespace>$(arg robot_namespace)</robotNamespace>
-      <updateRate>40</updateRate>
-      <bodyName>base_link</bodyName>
-      <frameId>base_link</frameId>
-      <topicName>navsat/fix</topicName>
-      <velocityTopicName>navsat/vel</velocityTopicName>
-      <referenceLatitude>$(optenv GAZEBO_WORLD_LAT 49.9)</referenceLatitude>
-      <referenceLongitude>$(optenv GAZEBO_WORLD_LON 8.9)</referenceLongitude>
-      <referenceHeading>90</referenceHeading>
-      <referenceAltitude>0</referenceAltitude>
-      <drift>0.0001 0.0001 0.0001</drift>
-    </plugin>
-  </gazebo>
   <!-- Optional custom includes. -->
   <xacro:include filename="$(arg urdf_extras)" />
   <!-- Optional for Clearpath internal softwares -->
   <xacro:include filename="$(arg cpr_urdf_extras)" />
+    <!-- Gazebo GPS Sensor (Hector plugin) -->
+    <gazebo>
+      <plugin name="gps_plugin" filename="libhector_gazebo_ros_gps.so">
+        <bodyName>gps_link</bodyName>
+        <frameId>gps_link</frameId>
+        <topicName>/gps/fix</topicName>
+        <velocityTopicName>/gps/fix_velocity</velocityTopicName>
+        <!-- 필수 참조 위치 (현실 위도/경도 기준) -->
+        <referenceLatitude>35.8475</referenceLatitude>
+        <referenceLongitude>127.1290</referenceLongitude>
+        <referenceAltitude>50.0</referenceAltitude>
+        <referenceHeading>0.0</referenceHeading>
+        <!-- 토픽이 나오게 만드는 핵심 요소 -->
+        <status>0</status>
+        <service>1</service>
+        <!-- 센서 속도 (10Hz = 100ms) -->
+        <updateRate>10</updateRate>
+      </plugin>
+    </gazebo>
 </robot>
